File: hardware/channel-card/level.kicad_sch (KiCad schematic)
At the start: 63 parts, among them SW201 MUTE (latching), SW202 DUCK (latching), U201 SSI2162, U202 NE5532, U203 NE5532, U204 OPA2171, U205 TL072, U206 DG413DY

Commit message: Channel card: mechanical parts, decisions 110-117
- 110 LM317/LM337 in D2PAK on copper (onsemi, LCSC)
- 111 SMD electrolytics <= 5.4 mm (ROQANG, Panasonic bipolar)
- 112 trimmers and jumper headers on the underside, bottom cover for /system
- 113 low-cut caps C0G 1206
- 114 pot shaft standard T18 15 mm; 115 trim stage scaled to 100k, pots chosen
  (blocked until RoHS declarations)
- 116 RoHS strict for every part and board (process)
- 117 button LED colours (JLCPCB basic 0805), Wurth chain headers
- J181 drawn as Thonkiconn 3.5 mm (pending /system), fields and footprints set,
  five sheets rebuilt, netlists match, ERC 0/0
- STATUS: seven For /system items (CV jack, 0805 meter bezel, panel screws,
  bottom cover, underside keep-out, RoHS invariant, contract doc updates)

Co-Authored-By: Claude Opus 5.5 <noreply@anthropic.com>
Parts:
- C221, C271: footprint Capacitor_THT:C_Radial_D5.0mm_H11.0mm_P2.00mm -> Capacitor_SMD:C_Elec_6.3x5.4; MPN (none) -> EEE-1VA100NP; Manufacturer (none) -> Panasonic; ProjectPN SX-C-003 -> SX-C-023; Supplier (none) -> Mouser; SupplierPN (none) -> 667-EEE-1VA100NP
- D203: MPN (none) -> NCD0805R1; Manufacturer (none) -> Foshan NationStar; ProjectPN SX-D-002 -> SX-D-015; Supplier (none) -> LCSC; SupplierPN (none) -> C84256
- D204: MPN (none) -> KT-0805G; Manufacturer (none) -> Hubei KENTO; ProjectPN SX-D-002 -> SX-D-011; Supplier (none) -> LCSC; SupplierPN (none) -> C2297
