File: hardware/channel-card/meter.kicad_sch (KiCad schematic)
At the start: 55 parts, among them U401 TL072, U402 TL072, U403 TL072, U404 TL072, U405 LM339, U406 LM339

Commit message: Add test pads to the channel card sheets
24 bare 1.5 mm test pads on key audio, control and ground nets across
the Input, Filter, Level, Routing and Meter sheets, named by net and
kept out of the BOM (decision 77). Each pad is in the reference
netlists, so the checks prove it sits on the intended net.

Co-Authored-By: Claude Opus 5.5 <noreply@anthropic.com>
Parts:
- added TP401: MV, TestPoint:TestPoint_Pad_D1.5mm, symbol Connector:TestPoint
Connections:
- net MV: now also TP401.1

Commit message: Channel card: meter LEDs 0805, op amp power levers (decision 123), RoHS audit
- Meter D411-D418 to 0805 LEDs (KT-0805G, KT-0805Y, NCD0805R1; decision 119)
- U107 NE5532 -> TL072; meter U401/U404 TL072 -> TL062CDR (SX-IC-024)
- Card load 113 / 95 mA typical, sizing 174 / 142 mA; netlists match, ERC 0/0
- RoHS audit of parts.csv (decision 122): 47 rows sourced; gaps SSI2144,
  SSI2162, AS3046D; THAT1646S08-U and ERA-V33J102V end of life at Mouser
  (docs/reviews/2026-10-09-rohs-audit.md); four rows requoted

Co-Authored-By: Claude Opus 5.5 <noreply@anthropic.com>
Parts:
- removed U401, U404: TL072, Package_SO:SOIC-8_3.9x4.9mm_P1.27mm, symbol Amplifier_Operational:TL072
- added U401, U404: TL062, Package_SO:SOIC-8_3.9x4.9mm_P1.27mm, symbol Amplifier_Operational:TL062
- D411, D412, D413, D414, D415: footprint LED_THT:LED_D3.0mm -> LED_SMD:LED_0805_2012Metric; MPN (none) -> KT-0805G; Manufacturer (none) -> Hubei KENTO; ProjectPN SX-D-004 -> SX-D-011; Supplier (none) -> LCSC; SupplierPN (none) -> C2297
- D416, D417: footprint LED_THT:LED_D3.0mm -> LED_SMD:LED_0805_2012Metric; MPN (none) -> KT-0805Y; Manufacturer (none) -> Hubei KENTO; ProjectPN SX-D-005 -> SX-D-016; Supplier (none) -> LCSC; SupplierPN (none) -> C2296
- D418: footprint LED_THT:LED_D3.0mm -> LED_SMD:LED_0805_2012Metric; MPN (none) -> NCD0805R1; Manufacturer (none) -> Foshan NationStar; ProjectPN SX-D-006 -> SX-D-015; Supplier (none) -> LCSC; SupplierPN (none) -> C84256
Connections:
- net +15V: now also U401.8 (V+), U404.8 (V+)
- net -15V: now also U401.4 (V-), U404.4 (V-)
- net AGND: now also U401.3 (+), U401.5 (+), U404.5 (+)
- net MV: now also U404.1, U404.2 (-)
- net at C401.1, R405.2, R406.2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: now also U404.3 (+)
- net at R402.2, U402.5 (+): now also U401.1
- net at R403.2, R404.1: now also U401.6 (-)
- net at R401.2, R402.1: now also U401.2 (-)
- net at R404.2, U403.5 (+): now also U401.7
- new net: U404.6 (-), U404.7

Commit message: Channel card: fee-free TL072CDT, 78L05G-AB3-R, BZT52C6V2, UNI-ROYAL resistors (decision 137)
SX-IC-007 TL072 -> ST TL072CDT (LCSC C6961, basic), SX-IC-012 78L05 -> UTC
78L05G-AB3-R (C71136, basic; pins 1 O 2 G 3 I, not the -AB3-C-R variant),
SX-D-001 -> hongjiacheng BZT52C6V2 (C19077403, preferred), SX-R-011/036/042
-> UNI-ROYAL 0805W8F (preferred). Datasheet facts and RoHS sources in
parts.csv. Filter, level, meter and chain sheets rebuilt: netlists match,
ERC 0/0. costs.py extended: 82 -> 80 fee types. Master STATUS notes that
its TL072 symbols still need the ST fields.

Co-Authored-By: Claude Opus 5.5 <noreply@anthropic.com>
Parts:
- U402, U403: MPN (none) -> TL072CDT; Manufacturer Texas Instruments -> STMicroelectronics; Supplier (none) -> LCSC; SupplierPN (none) -> C6961

Commit message: Channel card: cost levers (decisions 139-143)
- U303 DG412 -> DG413, SC send on the NC section (139)
- All values E24 with JLCPCB fee-free parts; E24 pairs for V/oct
  and fader law, meter ladder re-fitted (140)
- Filter temperature compensation to the backlog (141)
- MUTE/DUCK switched by the buttons' spare pole, U206 DG413 removed;
  100k hold resistors, no dependence on contact sequence (142)
- TL072 difference receiver with 10k 0.1 % instead of the AD8273 (143)
- Trimmers from Mouser, CUTOFF pot from Tayda A-4730
- Breadboard tests 11 (X5R coupling caps) and 12 (fixed V/oct)
- costs.py estimate, 4 channels: EUR 1,035 -> 946

Co-Authored-By: Claude Opus 5.5 <noreply@anthropic.com>
Parts:
- R410: value 19k1 -> 39k; ProjectPN SX-R-037 -> SX-R-104
- R411: value 4k02 -> 8k2; ProjectPN SX-R-038 -> SX-R-105
- R412: value 2k -> 3k9; ProjectPN SX-R-003 -> SX-R-099
- R413: value 1k43 -> 3k; ProjectPN SX-R-039 -> SX-R-063
- R414: value 1k54 -> 3k; ProjectPN SX-R-040 -> SX-R-063
- R415: value 845 -> 1k8; ProjectPN SX-R-041 -> SX-R-101
- R416: value 750 -> 1k5; ProjectPN SX-R-042 -> SX-R-044
- R417: value 237 -> 470; ProjectPN SX-R-043 -> SX-R-055
- R418: value 110 -> 220; ProjectPN SX-R-022 -> SX-R-106
