File: hardware/channel-card/routing.kicad_sch (KiCad schematic)
At the start: 39 parts, among them J301 AUX1 PRE 1-3/2-4, POST 3-5/4-6, J302 AUX2 PRE 1-3/2-4, POST 3-5/4-6, Q301 MMBT3904, SW301 PFL (latching), SW302 SC SEND (latching), SW303 COMP BUS (latching), U301 NE5532, U302 DG413DY, U303 DG412DY

Commit message: Channel card: cost levers (decisions 139-143)
- U303 DG412 -> DG413, SC send on the NC section (139)
- All values E24 with JLCPCB fee-free parts; E24 pairs for V/oct
  and fader law, meter ladder re-fitted (140)
- Filter temperature compensation to the backlog (141)
- MUTE/DUCK switched by the buttons' spare pole, U206 DG413 removed;
  100k hold resistors, no dependence on contact sequence (142)
- TL072 difference receiver with 10k 0.1 % instead of the AD8273 (143)
- Trimmers from Mouser, CUTOFF pot from Tayda A-4730
- Breadboard tests 11 (X5R coupling caps) and 12 (fixed V/oct)
- costs.py estimate, 4 channels: EUR 1,035 -> 946

Co-Authored-By: Claude Opus 5.5 <noreply@anthropic.com>
Parts:
- removed U303: DG412DY, Package_SO:SOIC-16_3.9x9.9mm_P1.27mm, symbol Analog_Switch:DG412xY
- added U303: DG413DY, Package_SO:SOIC-16_3.9x9.9mm_P1.27mm, symbol Analog_Switch:DG413xY
- R305, R306: value 44k2 -> 47k; ProjectPN SX-R-034 -> SX-R-032
Connections:
- net +15V: now also U303.13 (V+)
- net +5V: now also U303.12 (VL)
- net -15V: now also U303.4 (V-)
- net AGND: now also U303.10, U303.11, U303.5 (GND), U303.9
- net CUE_L: now also U303.3
- net CUE_R: now also U303.7
- net PFL_CTRL: now also U303.1, U303.8
- net SC: now also U303.14
- net at R305.2, R306.2: now also U303.15
- net at R304.2: now also U303.6
- net at R303.2: now also U303.2
- net SC_OFF: now reaches SW302.1 (A)
- net SC_OFF: now also R315.2, U303.16
- net SC_CTRL: no longer names the net of SW302.3 (C)
- net SC_CTRL: no longer R315.2

Commit message: Buttons: SX-SW-001 is the latching GPBS850L, not the momentary GPBS850N
Electrokit 41012905 (on-on, latching) links the GPBS850N datasheet, which
is the momentary twin (Electrokit 41015527, Mouser "Non-Latching ON-(ON)");
the MPN was copied from that file. The latching part is CW GPBS850L
(datasheet Rev 2, 2014: same body, pin grid and pressed = 2-3, 5-6 contacts;
plunger 4.0 mm instead of 3.8).

MPN and footprint name corrected on all 17 button symbols, the generator
scripts and the input reference; parts.csv gets the GPBS850L datasheet and
RoHS source (Mouser 629-GPBS-850L, DigiKey CW179-ND); prices.csv gets the
Electrokit price (6.48 SEK ex VAT at 25+). Erratum on decision 75, checklist
item for the delivered switches and cap sizing, correction notes in the
RoHS audit and the cost review. No wiring change; ERC 0/0 on both cards.
Estimate €769 / €1,037 / €1,609 for 4 / 8 / 16 channels.

Co-Authored-By: Claude Opus 5.5 <noreply@anthropic.com>
Parts:
- SW301, SW302, SW303: footprint syntsamix:SW_Latching_8.5x8.5mm_CW_GPBS850N -> syntsamix:SW_Latching_8.5x8.5mm_CW_GPBS850L; MPN GPBS850N -> GPBS850L
Changed lines of the file:
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@@
 			)
 		)
-		(property "Footprint" "syntsamix:SW_Latching_8.5x8.5mm_CW_GPBS850N"
+		(property "Footprint" "syntsamix:SW_Latching_8.5x8.5mm_CW_GPBS850L"
 			(at 233.68 279.4 0)
 			(hide yes)
@@
 			)
 		)
-		(property "MPN" "GPBS850N"
+		(property "MPN" "GPBS850L"
 			(at 233.68 279.4 0)
 			(hide yes)
@@
 			)
 		)
-		(property "Footprint" "syntsamix:SW_Latching_8.5x8.5mm_CW_GPBS850N"
+		(property "Footprint" "syntsamix:SW_Latching_8.5x8.5mm_CW_GPBS850L"
 			(at 40.64 279.4 0)
 			(hide yes)
@@
 			)
 		)
-		(property "MPN" "GPBS850N"
+		(property "MPN" "GPBS850L"
 			(at 40.64 279.4 0)
 			(hide yes)
@@
 			)
 		)
-		(property "Footprint" "syntsamix:SW_Latching_8.5x8.5mm_CW_GPBS850N"
+		(property "Footprint" "syntsamix:SW_Latching_8.5x8.5mm_CW_GPBS850L"
 			(at 137.16 279.4 0)
 			(hide yes)
@@
 			)
 		)
-		(property "MPN" "GPBS850N"
+		(property "MPN" "GPBS850L"
 			(at 137.16 279.4 0)
 			(hide yes)

Commit message: Channel card: CD4052B bus assign, PFL and SC send switches at the virtual-earth bus ends, LCSC BOCHEN trimmers (decisions 183-184)
Co-Authored-By: Claude Opus 5.5 <noreply@anthropic.com>
Parts:
- removed U302, U303: DG413DY, Package_SO:SOIC-16_3.9x9.9mm_P1.27mm, symbol Analog_Switch:DG413xY
- added C307, C308: 100n, Capacitor_SMD:C_0805_2012Metric, symbol Device:C
- added U302, U303, U304: CD4052B, Package_SO:SOIC-16_3.9x9.9mm_P1.27mm, symbol Analog_Switch:HEF4052BT
Connections:
- net +15V: no longer C303.1, C305.1
- net +5V: now also C303.1, C305.1, C307.1, U302.16 (VDD), U303.16 (VDD), U304.16 (VDD)
- net -15V: no longer C304.1, C306.1
- net AGND: now also C307.2, C308.2, U302.6 (~{E}), U302.8 (VSS), U302.9 (S2), U303.1 (2Y0), U303.12 (1Y0), U303.6 (~{E}), U303.8 (VSS), U303.9 (S2), U304.14 (1Y1), U304.6 (~{E}), U304.8 (VSS), U304.9 (S2)
- net COMP_CTRL: now also U302.10 (S1)
- net COMP_L: now also U302.14 (1Y1)
- net COMP_R: now also U302.5 (2Y1)
- net CUE_L: now also U303.14 (1Y1)
- net CUE_R: now also U303.5 (2Y1)
- net MAIN_L: now also U302.12 (1Y0)
- net MAIN_R: now also U302.1 (2Y0)
- net PFL_CTRL: now also U303.10 (S1)
- net SC: now also U304.12 (1Y0)
- net SC_OFF: now also U304.10 (S1)
- net at R301.2: now also U302.13 (1Z)
- net at R305.2, R306.2: now also U304.13 (1Z)
- net at R302.2: now also U302.3 (2Z)
- net at R303.2: now also U303.13 (1Z)
- net at R304.2: now also U303.3 (2Z)
- new net VEE: C304.1, C306.1, C308.1, U302.7 (VEE), U303.7 (VEE), U304.7 (VEE)
- no-connect marks 6 -> 21
