File: hardware/master/aux_sends.kicad_sch (KiCad schematic)
At the start: 43 parts, among them J601 AUX1 SEND L/MONO, J602 AUX1 SEND R, J621 AUX2 SEND L/MONO, J622 AUX2 SEND R, U601 NE5532, U621 NE5532, U641 DG411DY

Commit message: System: cost review and cost control (decisions 132-137)
Rean NYS216 jacks with a new footprint (132), through-hole parts hand-soldered (133), E24 values owned per board (134), live-device cost principle (135), /cost with the cost-controller sub-agent, tools/costs.py and a private ledger of realized costs (136), JLCPCB fee-free parts first (137).

Co-Authored-By: Claude Opus 5.5 <noreply@anthropic.com>
Parts:
- J601, J602, J621, J622: footprint Connector_Audio:Jack_6.35mm_Neutrik_NMJ6HCD2_Horizontal -> syntsamix:Jack_6.35mm_Rean_NYS216_Horizontal; MPN NMJ6HCD2 -> NYS216; Manufacturer Neutrik -> Rean; ProjectPN SX-CONN-001 -> SX-CONN-015
Changed lines of the file:
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@@
 			)
 		)
-		(property "Footprint" "Connector_Audio:Jack_6.35mm_Neutrik_NMJ6HCD2_Horizontal"
+		(property "Footprint" "syntsamix:Jack_6.35mm_Rean_NYS216_Horizontal"
 			(at 190.5 312.42 0)
 			(hide yes)
@@
 			)
 		)
-		(property "ProjectPN" "SX-CONN-001"
+		(property "ProjectPN" "SX-CONN-015"
 			(at 190.5 312.42 0)
 			(hide yes)
@@
 			)
 		)
-		(property "Manufacturer" "Neutrik"
+		(property "Manufacturer" "Rean"
 			(at 190.5 312.42 0)
 			(hide yes)
@@
 			)
 		)
-		(property "MPN" "NMJ6HCD2"
+		(property "MPN" "NYS216"
 			(at 190.5 312.42 0)
 			(hide yes)
@@
 			)
 		)
-		(property "Footprint" "Connector_Audio:Jack_6.35mm_Neutrik_NMJ6HCD2_Horizontal"
+		(property "Footprint" "syntsamix:Jack_6.35mm_Rean_NYS216_Horizontal"
 			(at 190.5 246.38 0)
 			(hide yes)
@@
 			)
 		)
-		(property "ProjectPN" "SX-CONN-001"
+		(property "ProjectPN" "SX-CONN-015"
 			(at 190.5 246.38 0)
 			(hide yes)
@@
 			)
 		)
-		(property "Manufacturer" "Neutrik"
+		(property "Manufacturer" "Rean"
 			(at 190.5 246.38 0)
 			(hide yes)
@@
 			)
 		)
-		(property "MPN" "NMJ6HCD2"
+		(property "MPN" "NYS216"
 			(at 190.5 246.38 0)
 			(hide yes)
@@
 			)
 		)
-		(property "Footprint" "Connector_Audio:Jack_6.35mm_Neutrik_NMJ6HCD2_Horizontal"
+		(property "Footprint" "syntsamix:Jack_6.35mm_Rean_NYS216_Horizontal"
 			(at 190.5 127 0)
 			(hide yes)
@@
 			)
 		)
-		(property "ProjectPN" "SX-CONN-001"
+		(property "ProjectPN" "SX-CONN-015"
 			(at 190.5 127 0)
 			(hide yes)
@@
 			)
 		)
-		(property "Manufacturer" "Neutrik"
+		(property "Manufacturer" "Rean"
 			(at 190.5 127 0)
 			(hide yes)
@@
 			)
 		)
-		(property "MPN" "NMJ6HCD2"
+		(property "MPN" "NYS216"
 			(at 190.5 127 0)
 			(hide yes)
@@
 			)
 		)
-		(property "Footprint" "Connector_Audio:Jack_6.35mm_Neutrik_NMJ6HCD2_Horizontal"
+		(property "Footprint" "syntsamix:Jack_6.35mm_Rean_NYS216_Horizontal"
 			(at 190.5 60.96 0)
 			(hide yes)
@@
 			)
 		)
-		(property "ProjectPN" "SX-CONN-001"
+		(property "ProjectPN" "SX-CONN-015"
 			(at 190.5 60.96 0)
 			(hide yes)
@@
 			)
 		)
-		(property "Manufacturer" "Neutrik"
+		(property "Manufacturer" "Rean"
 			(at 190.5 60.96 0)
 			(hide yes)
@@
 			)
 		)
-		(property "MPN" "NMJ6HCD2"
+		(property "MPN" "NYS216"
 			(at 190.5 60.96 0)
 			(hide yes)

Commit message: Master card: fee-free parts and E24 values (decisions 144, 146-150)
- 144: AUX return and master fader laws on the channel's E24 pairs
- 146: meter ladder on fee-free E24 values (0.45 mA, within 0.14 dB); R732 22k + R737 560R
- 147: compressor R420/R426 E24 pairs, GR LED ladder 470k/4k3, SC LPF C503 2 x 47n C0G
  (Q 0.707, 44-478 Hz); TL072 symbols ST TL072CDT
- 148: AUX return receivers TL072 difference amplifiers (AD8273 gone from the project)
- 149: R421 plain 1k; compressor temperature compensation to the backlog
- 150: DG413, SSI2162, DRV135UA, AS3046D hand-soldered on the prototype master
  (symbol field Assembly, read by tools/costs.py); SPOF noted in the backlog
- Part swaps: button LEDs per colour, D504 BAT54W, D705-D712 1N4007W SOD-123FL,
  U641 DG411 -> DG413 with a Q601 inverter for send 1 (emitter on PGND, invariant 4)
- 70 -> 38 extended/consigned SMD types (about EUR 193 -> 105 per order);
  estimate EUR 794 / 1,074 / 1,671 for 4 / 8 / 16 channels
- Docs: STATUS, CONTINUE-FROM-HERE, ROADMAP backlog, SPEC, hardware/CLAUDE.md lessons

Co-Authored-By: Claude Opus 5.5 <noreply@anthropic.com>
Parts:
- removed U641: DG411DY, Package_SO:SOIC-16_3.9x9.9mm_P1.27mm, symbol Analog_Switch:DG411xY
- added Q601: MMBT3904, Package_TO_SOT_SMD:SOT-23, symbol Transistor_BJT:Q_NPN_BEC
- added R612, R613: 100k, Resistor_SMD:R_0805_2012Metric, symbol Device:R
- added U641: DG413DY, Package_SO:SOIC-16_3.9x9.9mm_P1.27mm, symbol Analog_Switch:DG413xY
Connections:
- net +15V: now also U641.13 (V+)
- net +5V: now also R613.1, U641.12 (VL)
- net -15V: now also U641.4 (V-)
- net AGND: now also U641.5 (GND)
- net DET1: now also R612.1
- net DET2: now also U641.16, U641.9
- net at R601.2, R602.1, U601.2 (-): now also U641.2, U641.6
- net at R621.2, R622.1, U621.2 (-): now also U641.10, U641.15
- net at R603.1: now also U641.3
- net at R624.1: now also U641.14
- net at R623.1: now also U641.11
- net at R604.1: now also U641.7
- new net: Q601.1 (B), R612.2
- new net MONO1: Q601.3 (C), R613.2, U641.1, U641.8
- new net PGND: Q601.2 (E)

Commit message: Master: rear jacks on two 26-pin row-board ribbons (decision 163)
J603 (AUX sends sheet) carries main outs and both AUX sends to the
output row board; J903 (Power sheet) brings the AUX returns, SC EXT
and the ground-lift switch (pins 25/26) from the input row board.
Pairs with a ground between them; row boards hold only jacks, header
and SW901. Netlist checks 0 problems, ERC 0/0.

Co-Authored-By: Claude Opus 5.5 <noreply@anthropic.com>
Parts:
- removed J601: AUX1 SEND L/MONO, syntsamix:Jack_6.35mm_Rean_NYS216_Horizontal, symbol Connector_Audio:AudioJack3_Switch
- removed J602: AUX1 SEND R, syntsamix:Jack_6.35mm_Rean_NYS216_Horizontal, symbol Connector_Audio:AudioJack3_Switch
- removed J621: AUX2 SEND L/MONO, syntsamix:Jack_6.35mm_Rean_NYS216_Horizontal, symbol Connector_Audio:AudioJack3_Switch
- removed J622: AUX2 SEND R, syntsamix:Jack_6.35mm_Rean_NYS216_Horizontal, symbol Connector_Audio:AudioJack3_Switch
- added J603: REAR OUTPUTS, Connector_IDC:IDC-Header_2x13_P2.54mm_Vertical, symbol Connector_Generic:Conn_02x13_Odd_Even
Connections:
- net AGND: now also J603.1 (Pin_1), J603.10 (Pin_10), J603.13 (Pin_13), J603.16 (Pin_16), J603.19 (Pin_19), J603.21 (Pin_21), J603.23 (Pin_23), J603.24 (Pin_24), J603.25 (Pin_25), J603.26 (Pin_26), J603.4 (Pin_4), J603.7 (Pin_7)
- net DET1: now also J603.20 (Pin_20)
- net DET2: now also J603.22 (Pin_22)
- net L1_T: now reaches R607.2
- net L1_T: now also J603.8 (Pin_8)
- net R2_RING: now reaches R630.1
- net R2_RING: now also J603.18 (Pin_18)
- net R2_T: now reaches R629.2
- net R2_T: now also J603.17 (Pin_17)
- net L1_RING: now reaches R608.1
- net L1_RING: now also J603.9 (Pin_9)
- net R1_RING: now reaches R610.1
- net R1_RING: now also J603.12 (Pin_12)
- net L2_T: now reaches R627.2
- net L2_T: now also J603.14 (Pin_14)
- net R1_T: now reaches R609.2
- net R1_T: now also J603.11 (Pin_11)
- net L2_RING: now reaches R628.1
- net L2_RING: now also J603.15 (Pin_15)
- new net MAIN_L_COLD: J603.3 (Pin_3)
- new net MAIN_L_HOT: J603.2 (Pin_2)
- new net MAIN_R_COLD: J603.6 (Pin_6)
- new net MAIN_R_HOT: J603.5 (Pin_5)
- no-connect marks 10 -> 0
