File: hardware/master/sidechain.kicad_sch (KiCad schematic)
At the start: 69 parts, among them J501 SC EXT IN, Q501 MMBT3904, SW501 SC BUS (latching), SW502 SC LPF BYPASS (latching), SW503 SC LISTEN (latching), U501 TL072, U502 TL072, U503 TL072, U504 TL072, U505 TL072, U506 DG413DY, U507 DG413DY, U508 DG413DY

Commit message: Master card: draw decisions 97 and 98, OPA2171 fader-law stages (103), SC_ENV drive (104)
- AUX returns: SC_ENV into the summer's virtual earth through R232/R332 30k1,
  R233/R333 removed, summer + input on AGND (decision 97)
- Q501 emitter and button pull-downs R237/239/241, R337/339/341, R455,
  R523/525/527 to PGND (decision 98)
- U206, U306, U705 = OPA2171 for the pot buffer and control summer; superdiodes
  on the TL072s U207, U307, U706 (decision 103)
- Sidechain: DEPTH negative (R518 to -15 V), U505B follower fed back after R521,
  D504 BAT54T1G clamp to AGND (decision 104); simulation rerun with 1.7 kOhm load
- R421 on its 0603 footprint (system validation finding 3)
- Power budget, parts list, STATUS, decisions and working notes updated

Co-Authored-By: Claude Opus 5.5 <noreply@anthropic.com>
Parts:
- added D504: BAT54T1G, Diode_SMD:D_SOD-123, symbol Device:D
Connections:
- net +15V: no longer R518.2
- net -15V: now also R518.2
- net AGND: now also D504.1 (K); no longer Q501.2 (E), R523.1, R525.1, R527.1
- net PGND: now also Q501.2 (E), R523.1, R525.1, R527.1
- net SC_ENV: now also U505.6 (-), D504.2 (A)
- net at R521.1, U505.7: no longer U505.6 (-)

Commit message: Master card: DRV135 outputs, TL062 levers, SMD electrolytics, both raw rails watched (decisions 125-128)
/board master pre-layout session; the user delegated the open points.
- Confirms the [proposed] parts of decisions 89-94 (Q5 checked, +22 dB
  makeup kept for the breadboard, fallback R439 = 330k).
- 125: TI DRV135UA replaces the end-of-life THAT1646 (THAT memo
  2026-09-01); same SO-8 pinout, LCSC C544663.
- 126: U409, U410, U802, U804 TL072 -> TL062; superdiodes and U407 stay.
- 127: master electrolytics to SMD (decision 111 parts, 5.4 mm).
- 128: U707C watches -20V_RAW (22k6/100k), wired-OR with the +20 V trip.
- Würth fields on J101/J901, BAT54 LCSC C152458, G6K and header
  drawings checked, LCSC stock checked; budget 331/260 mA typical.
- parts.csv candidates for master pots and meter LEDs; lcsc_check.py
  handles MOhm.
ERC 0/0, all netlist checks 0 problems, reuse lint clean.

Co-Authored-By: Claude Opus 5.5 <noreply@anthropic.com>
Parts:
- D504: Supplier (none) -> LCSC; SupplierPN (none) -> C152458

Commit message: System: cost review and cost control (decisions 132-137)
Rean NYS216 jacks with a new footprint (132), through-hole parts hand-soldered (133), E24 values owned per board (134), live-device cost principle (135), /cost with the cost-controller sub-agent, tools/costs.py and a private ledger of realized costs (136), JLCPCB fee-free parts first (137).

Co-Authored-By: Claude Opus 5.5 <noreply@anthropic.com>
Parts:
- J501: footprint Connector_Audio:Jack_6.35mm_Neutrik_NMJ6HCD2_Horizontal -> syntsamix:Jack_6.35mm_Rean_NYS216_Horizontal; MPN NMJ6HCD2 -> NYS216; Manufacturer Neutrik -> Rean; ProjectPN SX-CONN-001 -> SX-CONN-015
Changed lines of the file:
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@@
 			)
 		)
-		(property "Footprint" "Connector_Audio:Jack_6.35mm_Neutrik_NMJ6HCD2_Horizontal"
+		(property "Footprint" "syntsamix:Jack_6.35mm_Rean_NYS216_Horizontal"
 			(at 30.48 109.22 0)
 			(hide yes)
@@
 			)
 		)
-		(property "ProjectPN" "SX-CONN-001"
+		(property "ProjectPN" "SX-CONN-015"
 			(at 30.48 109.22 0)
 			(hide yes)
@@
 			)
 		)
-		(property "Manufacturer" "Neutrik"
+		(property "Manufacturer" "Rean"
 			(at 30.48 109.22 0)
 			(hide yes)
@@
 			)
 		)
-		(property "MPN" "NMJ6HCD2"
+		(property "MPN" "NYS216"
 			(at 30.48 109.22 0)
 			(hide yes)

Commit message: Master card: SC LPF pot RV501 a standard Alpha dual B100K (decision 138)
The reverse-log dual 100k had no standard 9 mm T18 source. RV501 becomes
Alpha RD902F-40-15K-B100K-0057 (Thonk, SX-POT-015), RoHS cleared by
Alpha's general declaration. Same circuit; simulated sweep 46/60/85/146/510 Hz
at CCW/25 %/middle/75 %/CW. Other non-B master pots checked against Alpha's
0.02 W rating: all well under it. Netlist checks 0 problems, ERC 0/0.

Co-Authored-By: Claude Opus 5.5 <noreply@anthropic.com>
Parts:
- RV501: value SC LPF 100k rev. log dual -> SC LPF B100K dual; MPN (none) -> RD902F-40-15K-B100K-0057; Note Panel SC LPF: reverse-log (C) taper, CW = 510 Hz, CCW = 46 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 -> Panel SC LPF: linear (B) taper, CW = 510 Hz, middle 85 Hz, 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; ProjectPN SX-POT-008 -> SX-POT-015; Supplier (none) -> Thonk

Commit message: Master card: fee-free parts and E24 values (decisions 144, 146-150)
- 144: AUX return and master fader laws on the channel's E24 pairs
- 146: meter ladder on fee-free E24 values (0.45 mA, within 0.14 dB); R732 22k + R737 560R
- 147: compressor R420/R426 E24 pairs, GR LED ladder 470k/4k3, SC LPF C503 2 x 47n C0G
  (Q 0.707, 44-478 Hz); TL072 symbols ST TL072CDT
- 148: AUX return receivers TL072 difference amplifiers (AD8273 gone from the project)
- 149: R421 plain 1k; compressor temperature compensation to the backlog
- 150: DG413, SSI2162, DRV135UA, AS3046D hand-soldered on the prototype master
  (symbol field Assembly, read by tools/costs.py); SPOF noted in the backlog
- Part swaps: button LEDs per colour, D504 BAT54W, D705-D712 1N4007W SOD-123FL,
  U641 DG411 -> DG413 with a Q601 inverter for send 1 (emitter on PGND, invariant 4)
- 70 -> 38 extended/consigned SMD types (about EUR 193 -> 105 per order);
  estimate EUR 794 / 1,074 / 1,671 for 4 / 8 / 16 channels
- Docs: STATUS, CONTINUE-FROM-HERE, ROADMAP backlog, SPEC, hardware/CLAUDE.md lessons

Co-Authored-By: Claude Opus 5.5 <noreply@anthropic.com>
Parts:
- added C521: 47n C0G, Capacitor_SMD:C_0805_2012Metric, symbol Device:C
- C503: value 22n C0G -> 47n C0G; ProjectPN SX-C-017 -> SX-C-016
- D501: MPN (none) -> KT-0805G; Manufacturer (none) -> Hubei KENTO; ProjectPN SX-D-002 -> SX-D-011; Supplier (none) -> LCSC; SupplierPN (none) -> C2297
- D502: MPN (none) -> KT-0805W; Manufacturer (none) -> Hubei KENTO; ProjectPN SX-D-002 -> SX-D-017; Supplier (none) -> LCSC; SupplierPN (none) -> C34499
- D503: MPN (none) -> KT-0805Y; Manufacturer (none) -> Hubei KENTO; ProjectPN SX-D-002 -> SX-D-016; Supplier (none) -> LCSC; SupplierPN (none) -> C2296
- D504: value BAT54T1G -> BAT54W; MPN BAT54T1G -> BAT54W; Manufacturer onsemi -> hongjiacheng; SupplierPN C152458 -> C7502705
- RV501: Note Panel SC LPF: linear (B) taper, CW = 510 Hz, middle 85 Hz, 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 -> Panel SC LPF: linear (B) taper, CW = 478 Hz, middle 80 Hz, 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
- U501, U502, U503, U504, U505: MPN (none) -> TL072CDT; Manufacturer Texas Instruments -> STMicroelectronics; Supplier (none) -> LCSC; SupplierPN (none) -> C6961
- U506, U507, U508: Assembly (none) -> hand (decision 150)
Connections:
- net AGND: now also C521.2; no longer C503.2
- new net: C503.2, C521.1

Commit message: Buttons: SX-SW-001 is the latching GPBS850L, not the momentary GPBS850N
Electrokit 41012905 (on-on, latching) links the GPBS850N datasheet, which
is the momentary twin (Electrokit 41015527, Mouser "Non-Latching ON-(ON)");
the MPN was copied from that file. The latching part is CW GPBS850L
(datasheet Rev 2, 2014: same body, pin grid and pressed = 2-3, 5-6 contacts;
plunger 4.0 mm instead of 3.8).

MPN and footprint name corrected on all 17 button symbols, the generator
scripts and the input reference; parts.csv gets the GPBS850L datasheet and
RoHS source (Mouser 629-GPBS-850L, DigiKey CW179-ND); prices.csv gets the
Electrokit price (6.48 SEK ex VAT at 25+). Erratum on decision 75, checklist
item for the delivered switches and cap sizing, correction notes in the
RoHS audit and the cost review. No wiring change; ERC 0/0 on both cards.
Estimate €769 / €1,037 / €1,609 for 4 / 8 / 16 channels.

Co-Authored-By: Claude Opus 5.5 <noreply@anthropic.com>
Parts:
- SW501, SW502, SW503: footprint syntsamix:SW_Latching_8.5x8.5mm_CW_GPBS850N -> syntsamix:SW_Latching_8.5x8.5mm_CW_GPBS850L; MPN GPBS850N -> GPBS850L
Changed lines of the file:
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@@
 			)
 		)
-		(property "Footprint" "syntsamix:SW_Latching_8.5x8.5mm_CW_GPBS850N"
+		(property "Footprint" "syntsamix:SW_Latching_8.5x8.5mm_CW_GPBS850L"
 			(at 261.62 198.12 0)
 			(hide yes)
@@
 			)
 		)
-		(property "MPN" "GPBS850N"
+		(property "MPN" "GPBS850L"
 			(at 261.62 198.12 0)
 			(hide yes)
@@
 			)
 		)
-		(property "Footprint" "syntsamix:SW_Latching_8.5x8.5mm_CW_GPBS850N"
+		(property "Footprint" "syntsamix:SW_Latching_8.5x8.5mm_CW_GPBS850L"
 			(at 261.62 236.22 0)
 			(hide yes)
@@
 			)
 		)
-		(property "MPN" "GPBS850N"
+		(property "MPN" "GPBS850L"
 			(at 261.62 236.22 0)
 			(hide yes)
@@
 			)
 		)
-		(property "Footprint" "syntsamix:SW_Latching_8.5x8.5mm_CW_GPBS850N"
+		(property "Footprint" "syntsamix:SW_Latching_8.5x8.5mm_CW_GPBS850L"
 			(at 261.62 274.32 0)
 			(hide yes)
@@
 			)
 		)
-		(property "MPN" "GPBS850N"
+		(property "MPN" "GPBS850L"
 			(at 261.62 274.32 0)
 			(hide yes)

Commit message: Master: rear jacks on two 26-pin row-board ribbons (decision 163)
J603 (AUX sends sheet) carries main outs and both AUX sends to the
output row board; J903 (Power sheet) brings the AUX returns, SC EXT
and the ground-lift switch (pins 25/26) from the input row board.
Pairs with a ground between them; row boards hold only jacks, header
and SW901. Netlist checks 0 problems, ERC 0/0.

Co-Authored-By: Claude Opus 5.5 <noreply@anthropic.com>
Parts:
- removed J501: SC EXT IN, syntsamix:Jack_6.35mm_Rean_NYS216_Horizontal, symbol Connector_Audio:AudioJack3_Switch
Connections:
- net EXT_T: now reaches R506.1
- no-connect marks 7 -> 6
