File: hardware/master/meter.kicad_sch (KiCad schematic)
At the start: 103 parts, among them U801 TL072, U802 TL072, U803 TL072, U804 TL072, U805 LM339, U806 LM339, U807 LM339, U808 LM339, U809 LM339, U810 LM339

Commit message: Master card: DRV135 outputs, TL062 levers, SMD electrolytics, both raw rails watched (decisions 125-128)
/board master pre-layout session; the user delegated the open points.
- Confirms the [proposed] parts of decisions 89-94 (Q5 checked, +22 dB
  makeup kept for the breadboard, fallback R439 = 330k).
- 125: TI DRV135UA replaces the end-of-life THAT1646 (THAT memo
  2026-09-01); same SO-8 pinout, LCSC C544663.
- 126: U409, U410, U802, U804 TL072 -> TL062; superdiodes and U407 stay.
- 127: master electrolytics to SMD (decision 111 parts, 5.4 mm).
- 128: U707C watches -20V_RAW (22k6/100k), wired-OR with the +20 V trip.
- Würth fields on J101/J901, BAT54 LCSC C152458, G6K and header
  drawings checked, LCSC stock checked; budget 331/260 mA typical.
- parts.csv candidates for master pots and meter LEDs; lcsc_check.py
  handles MOhm.
ERC 0/0, all netlist checks 0 problems, reuse lint clean.

Co-Authored-By: Claude Opus 5.5 <noreply@anthropic.com>
Parts:
- removed U802, U804: TL072, Package_SO:SOIC-8_3.9x4.9mm_P1.27mm, symbol Amplifier_Operational:TL072
- added U802, U804: TL062, Package_SO:SOIC-8_3.9x4.9mm_P1.27mm, symbol Amplifier_Operational:TL062
Connections:
- net +15V: now also U802.8 (V+), U804.8 (V+)
- net -15V: now also U802.4 (V-), U804.4 (V-)
- net AGND: now also U802.3 (+), U804.3 (+)
- net MV_L: now also U802.6 (-), U802.7
- net MV_R: now also U804.6 (-), U804.7
- net at C801.1, R803.2, R804.2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: now also U802.5 (+)
- net at C802.1, R808.2, R809.2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: now also U804.5 (+)
- net at R802.2, U801.5 (+): now also U802.1
- net at R806.2, R807.1: now also U804.2 (-)
- net at R807.2, U803.5 (+): now also U804.1
- net at R801.2, R802.1: now also U802.2 (-)

Commit message: Master card: fee-free parts and E24 values (decisions 144, 146-150)
- 144: AUX return and master fader laws on the channel's E24 pairs
- 146: meter ladder on fee-free E24 values (0.45 mA, within 0.14 dB); R732 22k + R737 560R
- 147: compressor R420/R426 E24 pairs, GR LED ladder 470k/4k3, SC LPF C503 2 x 47n C0G
  (Q 0.707, 44-478 Hz); TL072 symbols ST TL072CDT
- 148: AUX return receivers TL072 difference amplifiers (AD8273 gone from the project)
- 149: R421 plain 1k; compressor temperature compensation to the backlog
- 150: DG413, SSI2162, DRV135UA, AS3046D hand-soldered on the prototype master
  (symbol field Assembly, read by tools/costs.py); SPOF noted in the backlog
- Part swaps: button LEDs per colour, D504 BAT54W, D705-D712 1N4007W SOD-123FL,
  U641 DG411 -> DG413 with a Q601 inverter for send 1 (emitter on PGND, invariant 4)
- 70 -> 38 extended/consigned SMD types (about EUR 193 -> 105 per order);
  estimate EUR 794 / 1,074 / 1,671 for 4 / 8 / 16 channels
- Docs: STATUS, CONTINUE-FROM-HERE, ROADMAP backlog, SPEC, hardware/CLAUDE.md lessons

Co-Authored-By: Claude Opus 5.5 <noreply@anthropic.com>
Parts:
- R811: value 115k -> 16k; ProjectPN SX-R-068 -> SX-R-005
- R812: value 13k3 -> 1k8; ProjectPN SX-R-069 -> SX-R-101
- R813: value 31k6 -> 4k7; ProjectPN SX-R-070 -> SX-R-004
- R814: value 22k6 -> 3k; ProjectPN SX-R-071 -> SX-R-063
- R815: value 16k2 -> 2k4; ProjectPN SX-R-072 -> SX-R-108
- R816: value 11k3 -> 1k5; ProjectPN SX-R-073 -> SX-R-044
- R817: value 8k06 -> 1k2; ProjectPN SX-R-074 -> SX-R-109
- R818: value 5k62 -> 750; ProjectPN SX-R-075 -> SX-R-042
- R819: value 5k11 -> 750; ProjectPN SX-R-076 -> SX-R-042
- R820: value 3k83 -> 510; ProjectPN SX-R-077 -> SX-R-110
- R821: value 2k15 -> 300; ProjectPN SX-R-078 -> SX-R-111
- R822: value 1k87 -> 270; ProjectPN SX-R-079 -> SX-R-112
- R823: value 866 -> 120; ProjectPN SX-R-080 -> SX-R-045
- U801, U803: MPN (none) -> TL072CDT; Manufacturer Texas Instruments -> STMicroelectronics; Supplier (none) -> LCSC; SupplierPN (none) -> C6961

Commit message: Master: headphone jack, 0805 LEDs, off-board parts in the estimate (decisions 169-171)
- J751 becomes a KK 1x3 header for the panel Rean NYS230 with a ready-made
  Molex 217797-1031 lead (169)
- Master meter, gain-reduction (yellow) and PFL-active LEDs all 0805 basic
  parts; SX-D-005/006 retired (170)
- tools/costs.py counts parts without a schematic symbol from
  docs/costs/offboard.csv, and the two rear row-board PCBs (171):
  estimate EUR 831 / 1,110 / 1,693 for 4 / 8 / 16 channels
- New parts SX-CONN-019..022; ready-made input-module cable noted for /system
- NYS216/NYS230 samples to order; heatsink choice on hold (none fits 25 mm
  at decision 167's 57 C air), options in master STATUS

Co-Authored-By: Claude Opus 5.5 <noreply@anthropic.com>
Parts:
- D805, D806, D807, D808, D809, D810, D811, D817, D818, D819, D820, D821, D822, D823: footprint LED_THT:LED_D3.0mm -> LED_SMD:LED_0805_2012Metric; MPN (none) -> KT-0805G; Manufacturer (none) -> Hubei KENTO; ProjectPN SX-D-004 -> SX-D-011; Supplier (none) -> LCSC; SupplierPN (none) -> C2297
- D812, D813, D814, D824, D825, D826: footprint LED_THT:LED_D3.0mm -> LED_SMD:LED_0805_2012Metric; MPN (none) -> KT-0805Y; Manufacturer (none) -> Hubei KENTO; ProjectPN SX-D-005 -> SX-D-016; Supplier (none) -> LCSC; SupplierPN (none) -> C2296
- D815, D816, D827, D828: footprint LED_THT:LED_D3.0mm -> LED_SMD:LED_0805_2012Metric; MPN (none) -> NCD0805R1; Manufacturer (none) -> Foshan NationStar; ProjectPN SX-D-006 -> SX-D-015; Supplier (none) -> LCSC; SupplierPN (none) -> C84256
