File: hardware/master/bus.kicad_sch (KiCad schematic)
At the start: 48 parts, among them J101 AUDIO CHAIN, U101 NE5532, U102 NE5532, U103 NE5532, U104 NE5532, U105 NE5532, U106 NE5532

Commit message: Master card: DRV135 outputs, TL062 levers, SMD electrolytics, both raw rails watched (decisions 125-128)
/board master pre-layout session; the user delegated the open points.
- Confirms the [proposed] parts of decisions 89-94 (Q5 checked, +22 dB
  makeup kept for the breadboard, fallback R439 = 330k).
- 125: TI DRV135UA replaces the end-of-life THAT1646 (THAT memo
  2026-09-01); same SO-8 pinout, LCSC C544663.
- 126: U409, U410, U802, U804 TL072 -> TL062; superdiodes and U407 stay.
- 127: master electrolytics to SMD (decision 111 parts, 5.4 mm).
- 128: U707C watches -20V_RAW (22k6/100k), wired-OR with the +20 V trip.
- Würth fields on J101/J901, BAT54 LCSC C152458, G6K and header
  drawings checked, LCSC stock checked; budget 331/260 mA typical.
- parts.csv candidates for master pots and meter LEDs; lcsc_check.py
  handles MOhm.
ERC 0/0, all netlist checks 0 problems, reuse lint clean.

Co-Authored-By: Claude Opus 5.5 <noreply@anthropic.com>
Parts:
- J101: MPN (none) -> 61203421621; Manufacturer (none) -> Wurth Elektronik; Note 34-pin shrouded keyed box header, pinout docs/CHAIN.md -> 34-pin shrouded keyed box header, pinout docs/CHAIN.md; und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; Supplier (none) -> Mouser; SupplierPN (none) -> 710-61203421621

Commit message: Master: back-to-back coupling pairs, ten NE5532 to TL072, Wakefield heatsinks, onsemi TO-220 regulators (decisions 172-174)
Co-Authored-By: Claude Opus 5.5 <noreply@anthropic.com>
Parts:
- removed U106: NE5532, Package_SO:SOIC-8_3.9x4.9mm_P1.27mm, symbol Amplifier_Operational:NE5532
- added U106: TL072, Package_SO:SOIC-8_3.9x4.9mm_P1.27mm, symbol Amplifier_Operational:TL072
Connections:
- net +15V: now also U106.8 (V+)
- net -15V: now also U106.4 (V-)
- net AGND: now also U106.3 (+), U106.5 (+)
- net SC: now also U106.2 (-)
- net SC_SUM: now also U106.1
- new net: U106.6 (-), U106.7
