File: hardware/master/aux_return1.kicad_sch (KiCad schematic)
At the start: 110 parts, among them J203 GAIN: fitted -6 dB (PRO), ope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, SW201 RETURN 1 MUTE (latching), SW202 RETURN 1 DUCK (latching), SW203 RETURN 1 COMP (latching), U201 TL072, U202 TL072, U203 SSI2162, U204 TL072, U205 TL072, U206 OPA2171, U207 TL072, U208 DG413DY, U209 DG413DY

Commit message: Master: AUX return MUTE and DUCK on the buttons, U208/U308 DG413 removed; checklists brought to decisions 174-175; decision 147 confirmed (decision 177)
Co-Authored-By: Claude Opus 5.5 <noreply@anthropic.com>
Parts:
- removed C232, C233: 100n, Capacitor_SMD:C_0805_2012Metric, symbol Device:C
- removed U208: DG413DY, Package_SO:SOIC-16_3.9x9.9mm_P1.27mm, symbol Analog_Switch:DG413xY
Connections:
- net +5V: no longer SW201.2 (B), SW202.2 (B)
- net -15V: now also SW201.3 (C)
- net AGND: now also R237.1, R239.1
- net DUCK_V: now also R239.2, SW202.2 (B)
- net MUTE_V: now also R237.2, SW201.2 (B)
- net PGND: no longer R237.1, R239.1
- net SC_ENV: now also SW202.3 (C)
- removed net DUCK_CTRL: R239.2, SW202.3 (C)
- removed net MUTE_CTRL: R237.2, SW201.3 (C)
