File: hardware/master/aux_return2.kicad_sch (KiCad schematic)
At the start: 110 parts, among them J303 GAIN: fitted -6 dB (PRO), ope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, SW301 RETURN 2 MUTE (latching), SW302 RETURN 2 DUCK (latching), SW303 RETURN 2 COMP (latching), U301 TL072, U302 TL072, U303 SSI2162, U304 TL072, U305 TL072, U306 OPA2171, U307 TL072, U308 DG413DY, U309 DG413DY

Commit message: Master: AUX return MUTE and DUCK on the buttons, U208/U308 DG413 removed; checklists brought to decisions 174-175; decision 147 confirmed (decision 177)
Co-Authored-By: Claude Opus 5.5 <noreply@anthropic.com>
Parts:
- removed C332, C333: 100n, Capacitor_SMD:C_0805_2012Metric, symbol Device:C
- removed U308: DG413DY, Package_SO:SOIC-16_3.9x9.9mm_P1.27mm, symbol Analog_Switch:DG413xY
Connections:
- net +5V: no longer SW301.2 (B), SW302.2 (B)
- net -15V: now also SW301.3 (C)
- net AGND: now also R337.1, R339.1
- net DUCK_V: now also R339.2, SW302.2 (B)
- net MUTE_V: now also R337.2, SW301.2 (B)
- net PGND: no longer R337.1, R339.1
- net SC_ENV: now also SW302.3 (C)
- removed net DUCK_CTRL: R339.2, SW302.3 (C)
- removed net MUTE_CTRL: R337.2, SW301.3 (C)
