File: hardware/power/power.kicad_pcb (KiCad board)
At the start: 2 copper layers, 177 x 35 mm, 91 parts, among them J101 24V IN, J102 POWER SW, J103 POWER LED, J401 MASTER, J402 CHAIN 1, Q101 SQJ457EP, Q102 SQJ457EP, U101 L78M05, U102 74HC14, U201 TPS54560, U301 TPS54560

Commit message: Power board: input EMI pi filter C108/L101 after Q102, PCB rebuilt (decision 187)
C108 4.7 uF 100 V on the brick side, L101 2.2 uH SRP7028A in series, then C103:
keeps the converters' 400 kHz input current off the brick lead (about -80 dB
against -44 dB in a hand model; L101 alone gains nothing because C101 resonates
with the lead near 400 kHz). No new part type. Input area re-placed (F101
upright, Q101/Q102 to the rear, VIN_PRE copper under L101); placement.py now
takes new parts and pad nets from the schematic. ERC 0/0, DRC 0, parity clean.

Co-Authored-By: Claude Opus 5.5 <noreply@anthropic.com>
Parts:
- added C108: 4u7 100V, Capacitor_SMD:C_1210_3225Metric, F.Cu at (93.0, 125.3)
- added L101: 2u2, Inductor_SMD:L_Bourns_SRP7028A_7.3x6.6mm, F.Cu at (96.4, 120.0)
- moved F101 11.2 mm to (65.5, 116.0), turned to 90 degrees
- moved Q101 8.70 mm to (78.3, 120.0)
- moved Q102 8.70 mm to (87.8, 120.0)
- moved TP102 7.78 mm to (72.6, 121.4)
- moved C102 6.71 mm to (97.6, 125.3), turned to 180 degrees
- turned C101 to 0 degrees
- turned D101 to 0 degrees
Connections:
- C102 pad 2: /VIN_SW -> /Input and clock/VIN_PRE
- Q102 pad 5: /VIN_SW -> /Input and clock/VIN_PRE
Routing:
- net Net-(C107-Pad1): track 29.9 -> 13.2 mm, vias 2 -> 0
- net PGND: track 126.3 -> 140.8 mm, vias 114 -> 108
- net /-20 V inverter/-20V_CONV: track 38.7 -> 46.6 mm, vias 37 -> 39
- net Net-(D302-A): track 17.6 -> 24.0 mm, vias 0 -> 2
- net /VIN_SW: track 79.5 -> 84.9 mm
- net Net-(U301-RT/CLK): track 27.1 -> 21.7 mm
- net Net-(D102-K): track 25.3 -> 29.3 mm, vias 0 -> 2
- net /Input and clock/VBRICK: track 26.8 -> 24.5 mm
- net Net-(D101-K): track 32.7 -> 34.8 mm
- net Net-(D302-K): track 28.9 -> 30.8 mm
- net Net-(C102-Pad1): track 2.14 -> 3.97 mm
- net Net-(U201-RT/CLK): track 14.3 -> 15.5 mm
- net /Input and clock/GATE: track 34.0 -> 32.8 mm, vias 2 -> 3
- net Net-(D202-A): track 22.7 -> 21.7 mm
- net Net-(U201-BOOT): track 5.22 -> 4.35 mm
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- added copper zone on F.Cu, net /Input and clock/VIN_PRE

Commit message: Power board: DNP switch-node RC snubber footprints across D201 and D301, bench EMI checklist (decision 189)
R208/C215 (SW to PGND, above D201) and R308/C315 (SW to -20V_CONV, beside
D301), 0805, not fitted: values from a bench measurement of the ringing on the
first boards ("Bench, first boards" in CHECKLISTS.md, with the input filter
check of decision 187). placement.py takes DNP and BOM flags from the symbols.
ERC 0/0, DRC 0, parity clean; cost unchanged.

Co-Authored-By: Claude Opus 5.5 <noreply@anthropic.com>
Parts:
- added C215: 470p 100V, Capacitor_SMD:C_0805_2012Metric, F.Cu at (128.8, 101.0)
- added C315: 470p 100V, Capacitor_SMD:C_0805_2012Metric, F.Cu at (137.6, 124.4)
- added R208: 4R7, Resistor_SMD:R_0805_2012Metric, F.Cu at (125.2, 101.0)
- added R308: 4R7, Resistor_SMD:R_0805_2012Metric, F.Cu at (135.5, 124.4)
Routing:
- net Net-(C107-Pad1): track 13.2 -> 29.9 mm, vias 0 -> 2
- net PGND: track 140.8 -> 124.9 mm, vias 108 -> 124
- net Net-(D302-A): track 24.0 -> 17.6 mm, vias 2 -> 0
- net Net-(U201-COMP): track 15.1 -> 19.3 mm
- net Net-(D201-K): track 14.9 -> 18.4 mm, vias 0 -> 2
- net /-20 V inverter/-20V_CONV: track 46.6 -> 49.5 mm
- net Net-(D101-K): track 34.8 -> 32.3 mm
- net Net-(C315-Pad1): track 0.00 -> 2.14 mm
- net Net-(U101-VO): track 26.2 -> 24.1 mm
- net Net-(C215-Pad1): track 0.00 -> 1.74 mm
- net Net-(D301-K): track 33.1 -> 34.7 mm
- net Net-(D202-A): track 21.7 -> 20.3 mm, vias 3 -> 2
- net /Input and clock/GATE: track 32.8 -> 31.5 mm
- net Net-(D302-K): track 30.8 -> 31.7 mm
- net Net-(J103-Pin_1): track 12.4 -> 11.7 mm
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
Commit message: Power board: EMI layout review, smaller switch-node copper, bottom-plane keep-outs under the hot loops
Switch-node pours cut to the pads plus a strip (buck about 95 to 71 mm2,
inverter about 149 to 98 mm2); the buck boot capacitor's switch-node link and
the MOSFET source link moved from the bottom to the top; bottom-layer track
keep-outs under the buck loop, the input filter, left of and below the
inverter's loop. Under the inverter IC the EN, RT/CLK and FB hops remain.
DRC 0 violations, 0 unconnected, schematic parity.

Co-Authored-By: Claude Opus 5.5 <noreply@anthropic.com>
Routing:
- net /-20 V inverter/-20V_CONV: track 49.5 -> 34.9 mm, vias 39 -> 37
- net /Input and clock/GATE: track 31.5 -> 44.3 mm, vias 3 -> 4
- net /+20V_RAW: track 71.6 -> 84.2 mm
- net Net-(D301-K): track 34.7 -> 45.5 mm
- net Net-(U301-EN): track 18.4 -> 27.7 mm
- net Net-(U301-RT/CLK): track 21.7 -> 30.2 mm
- net Net-(D302-K): track 31.7 -> 39.8 mm
- net Net-(U201-COMP): track 19.3 -> 25.0 mm
- net Net-(D202-K): track 16.0 -> 12.8 mm
- net PGND: track 124.9 -> 127.5 mm, vias 124 -> 123
- net Net-(U101-VO): track 24.1 -> 26.0 mm
- net Net-(D202-A): track 20.3 -> 22.0 mm, vias 2 -> 3
- net Net-(J102-Pin_1): track 12.7 -> 11.0 mm
- net Net-(D101-K): track 32.3 -> 30.7 mm
- net Net-(D302-A): track 17.6 -> 18.9 mm, vias 0 -> 2
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
Commit message: Power board: inverter control corner reworked, boot capacitor above the IC, compensation below it
C308 between pins 1 and 8 above U301 removes the BOOT hop and the switch-node
run round the IC; R303/C305/C306 and C304 below the IC remove the COMP hop;
the band below the inverter IC is clear of bottom tracks. EN, RT/CLK and FB
still cross the island under the IC (about 26 mm, from 55). A top PGND sliver
between C314's pads is covered by the inverter-output ground area. DRC 0
violations, 0 unconnected, schematic parity; reviewed by the user.

Co-Authored-By: Claude Opus 5.5 <noreply@anthropic.com>
Parts:
- moved C305 11.2 mm to (121.8, 132.6), turned to 0 degrees
- moved C308 10.6 mm to (121.0, 122.6)
- moved R303 10.00 mm to (121.8, 130.5), turned to 180 degrees
- moved C306 9.60 mm to (125.2, 130.5), turned to 180 degrees
- moved C304 3.30 mm to (118.3, 130.5)
Routing:
- net Net-(D301-K): track 45.5 -> 29.6 mm
- net Net-(U301-EN): track 27.7 -> 15.0 mm
- net /+20V_RAW: track 84.2 -> 71.6 mm
- net Net-(U201-COMP): track 25.0 -> 36.7 mm, vias 3 -> 4
- net Net-(D302-K): track 39.8 -> 28.4 mm, vias 3 -> 2
- net Net-(U301-RT/CLK): track 30.2 -> 18.9 mm
- net Net-(U301-BOOT): track 11.0 -> 3.19 mm, vias 2 -> 0
- net /Input and clock/GATE: track 44.3 -> 38.3 mm
- net /VIN_SW: track 84.3 -> 78.5 mm
- net Net-(U301-COMP): track 14.6 -> 10.8 mm, vias 2 -> 0
- net /Outputs/+20V_C1: track 13.7 -> 11.1 mm
- net PGND: track 127.5 -> 129.7 mm, vias 123 -> 125
- net Net-(D202-K): track 12.8 -> 14.8 mm
- net Net-(U101-VO): track 26.0 -> 27.8 mm
- net Net-(D202-A): track 22.0 -> 23.6 mm
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